File: cc2650_usb.kicad_pcb (KiCad board)
At the start: 2 copper layers, 49.9 x 28 mm, 147 parts, among them P1 CONN_01X07, P2 CONN_01X04, P3 CONN_01X02, P4 CONN_01X08, P5 VBAT, Q1 FDN340P, SW1 RST, U1 CC2650F128RHB, U2 XC6206P332MR, X1 24Mhz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

Commit message: All components placed (preliminary)
Parts:
- moved U2 0.06 mm to (144.3, 111.2)
Changed lines of the file:
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@@
     (area 129.724999 85.624999 179.775001 113.775001)
     (thickness 1.6)
-    (drawings 20)
+    (drawings 22)
     (tracks 260)
     (zones 0)
@@
     (descr "Through hole pin header")
     (tags "pin header")
-    (fp_text reference P1 (at -0.42 -14.06 360) (layer F.SilkS)
+    (fp_text reference P1 (at -0.42 -14.06) (layer F.SilkS)
       (effects (font (size 1 1) (thickness 0.15)))
     )
@@
     (descr "Through hole pin header")
     (tags "pin header")
-    (fp_text reference P2 (at 1.15 -21.19 360) (layer F.SilkS)
+    (fp_text reference P2 (at 1.15 -21.19) (layer F.SilkS)
       (effects (font (size 1 1) (thickness 0.15)))
     )
@@
   )
   (module TO_SOT_Packages_SMD:SOT-23 (layer F.Cu)
-    (at 144.36 111.21 90)
+    (at 144.29822 111.22 90)
     (descr "SOT-23, Standard")
     (tags SOT-23)
@@
     )
   )
+  (gr_text - (at 164.79 103.45) (layer B.SilkS)
+    (effects (font (size 1.5 1.5) (thickness 0.3)) (justify mirror))
+  )
+  (gr_text + (at 139.19 103.23) (layer B.SilkS)
+    (effects (font (size 1 1) (thickness 0.15)) (justify mirror))
+  )
   (gr_text + (at 138.8 113) (layer F.SilkS)

Commit message: Fix ground plane, add more silkscreen
Parts:
- moved REF** 2.20 mm to (143.1, 89.6)
- moved R1 1.24 mm to (142.9, 91.5)
- moved P1 0.10 mm to (157.4, 87.7)
- moved P2 0.09 mm to (161.1, 87.7)
Routing:
- net /~SRST~: track 25.0 -> 26.2 mm
Other:
- board text added: "CC2650 Breakoutboard PCB Antenna 2016-09-18"
- board text added: "GND"
- board text added: "RST"
- board text added: "RX"
- board text added: "TCK"
- board text added: "TDI"
- board text added: "TDO"
- board text added: "TMS"
- board text added: "TX"
- board text added: "VDD"
- board text added: "~RST~"
